File: chip-to-olinuxino-lcd/olinuxino-chip-cape.sch (KiCad schematic (older format))
At the start: 4 parts, among them U1 LCD Olinuxino Connector, U13 LCD Connector, U14 Generic Connector

Commit message: rerouting
Signed-off-by: Maxime Ripard <maxime.ripard@free-electrons.com>
Connections:
- net TPX1 renamed TP_X-
- net TPX2 renamed TP_X+
- net TPY1 renamed TP_Y-
- net TPY2 renamed TP_Y+
Changed lines of the file:
@@
 PWM0
 Text Label 8150 3000 0    60   ~ 0
-TPX2
+TP_X+
 Text Label 8150 3100 0    60   ~ 0
-TPY2
+TP_Y+
 Text Label 6850 1500 2    60   ~ 0
 LCD_D18
@@
 LCD_PWR
 Text Label 6850 3000 2    60   ~ 0
-TPX1
+TP_X-
 Text Label 6850 3100 2    60   ~ 0
-TPY1
+TP_Y-
 Text Label 5250 2500 0    60   ~ 0
 GPIO0
@@
 GPIO1
 Text Label 3050 1800 0    60   ~ 0
-TPX2
+TP_X+
 Text Label 3050 1900 0    60   ~ 0
-TPY2
+TP_Y+
 Text Label 3050 2000 0    60   ~ 0
 PWM0
@@
 LCD_DE
 Text Label 1750 1800 2    60   ~ 0
-TPX1
+TP_X-
 Text Label 1750 1900 2    60   ~ 0
-TPY1
+TP_Y-
 Text Label 1750 2000 2    60   ~ 0
 LCD_D2

Commit message: turn the connector around, and reroute
Signed-off-by: Maxime Ripard <maxime.ripard@free-electrons.com>
Connections:
- net GND: now also U13.1 (P1); no longer U1.2 (P2), U1.4 (P4), U14.1 (P1)
- net GND2: now reaches U13.39 (P39)
- net GND2: now also U1.2 (P2), U1.4 (P4)
- no-connect marks 49 -> 48
Changed lines of the file:
@@
 	1    0    0    -1
 $EndComp
-Text Label 3950 1200 2    60   ~ 0
-GND
 Text Label 5250 1200 0    60   ~ 0
 5V
@@
 NoConn ~ 4200 2900
 NoConn ~ 4200 3000
-NoConn ~ 2000 3100
-NoConn ~ 2000 1200
 NoConn ~ 2000 1300
 Text Label 1750 1400 2    60   ~ 0
 3.3V
-Wire Wire Line
-	3950 1200 4200 1200
 Wire Wire Line
 	5250 1200 5000 1200
@@
 5V
 Text Label 8150 1200 0    60   ~ 0
-GND
+GND2
 Wire Wire Line
 	6850 1300 7100 1300
@@
 3.3V
 NoConn ~ 4200 3100
+Wire Wire Line
+	1750 1200 2000 1200
+Text Label 1750 1200 2    60   ~ 0
+GND
+NoConn ~ 4200 1200
+Wire Wire Line
+	1750 3100 2000 3100
+Text Label 1750 3100 2    60   ~ 0
+GND2
 $EndSCHEMATC
